File: hardware/KiCad/tracking system/tracking system.kicad_pcb (KiCad board)
At the start: 2 copper layers, 60 x 40 mm, 47 parts, among them J1 TP_SWD, J2 USB_C_Receptacle_PowerOnly_6P, J3 battery_conn, J5 GPS_Conn, J6 GSM_Conn, J7 OLED_conn, SW1 POWER_BTN, SW2 DIST_BTN, U1 STM32L476RETx, U2 TP4056-42-ESOP8, U3 ME6211C33M5, Y1 32kHz, Y2 8MHz

Commit message: continued placing components in PCB
Parts:
- J1: footprint Connector_PinHeader_2.54mm:PinHeader_1x02_P2.54mm_Vertical -> Connector_PinHeader_2.54mm:PinHeader_1x04_P2.54mm_Vertical
- J3: footprint Connector_PinHeader_2.54mm:PinHeader_1x04_P2.54mm_Vertical -> Connector_PinHeader_2.54mm:PinHeader_1x02_P2.54mm_Vertical
- moved Y2 101.4 mm to (118.8, 100.2), turned to 90 degrees
- moved Y1 101.4 mm to (119.0, 93.5)
- moved C15 93.3 mm to (121.8, 94.8), turned to -90 degrees
- moved C12 90.6 mm to (121.5, 101.0), turned to -90 degrees
- moved C13 90.3 mm to (121.5, 98.0), turned to 90 degrees
- moved C14 90.2 mm to (121.8, 92.0), turned to 90 degrees
- moved SW2 89.8 mm to (125.2, 114.2)
- moved SW1 89.7 mm to (125.2, 108.0)
- moved J7 82.4 mm to (128.5, 84.5), turned to 90 degrees
- moved C11 81.0 mm to (130.8, 91.8), turned to 90 degrees
- moved R1 80.5 mm to (123.5, 99.2), turned to -90 degrees
- moved C9 79.9 mm to (132.5, 98.0), turned to -90 degrees
- moved C10 79.3 mm to (132.5, 91.8), turned to 90 degrees
- moved C7 78.4 mm to (130.8, 103.3), turned to 90 degrees
- moved C8 77.8 mm to (137.5, 109.0), turned to 180 degrees
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Routing:
- added copper zone on F.Cu, net GND
